File: nu-pogodi-pcb.kicad_sch (KiCad schematic)
At the start: 25 parts, among them J1 Pico_Socket_A, J2 Pico_Socket_B, J3 MSP2806 Socket A, J4 MSP2806 Socket B, J5 Conn_01x02_Pin, Q1 2N2222, SW1 SPST-NO 6x6mm, SW10 SW_DPDT_x2, SW2 SPST-NO 6x6mm, SW3 SPST-NO 6x6mm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

Commit message: Fixed pinout
Connections:
- net ROW_1: now also J1.10 (GPIO7); no longer J1.9 (GPIO6)
- net ROW_2: now also J1.9 (GPIO6); no longer J1.10 (GPIO7)
Changed lines of the file:
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@@
 		)
 	)
-	(label "ROW_1"
+	(label "ROW_2"
 		(at 111.76 59.69 0)
 		(effects
@@
 		)
 	)
-	(label "ROW_2"
+	(label "ROW_1"
 		(at 111.76 62.23 0)
 		(effects
